File: CoolCubeLM1875kicad_pro/CoolCubeLM1875kicad_pro.kicad_pcb (KiCad board)
At the start: 2 copper layers, 120 x 168.9 mm, 199 parts, among them IC2 RESET, IC3 TPS7A2033, IC4 ESP32-Wrover-IE-N16R8, IC5 BOOT, IC6 LM1971, IC7 TPS7A4901, J1 AC, J10 LOW OUT, J2 AC, J3 GND, J4 SYSTEM CONNECTOR, J5 GND, J6 GND, J7 HI OUT, J8 PROG, J9 GND, K1 Relay_DPST-NO, K2 STBY RELAY, Q2 BD140, Q3 BC549, Q4 BC559, Q5 BC549, U1 LM1875, U10 OPA171, U2 LM1875, U3 LMR51430, U4 PCM5102A, U5 OPA1656ID, U6 AMS1117-3.3, U7 TPS7A39, U8 ATtiny1614, U9 MCP6H01

Commit message: more work
Parts:
- removed C1, C7: 1uF, Capacitor_THT:C_Rect_L7.5mm_W6.5mm_P5.00mm
- removed the J8 at (195.4, 77.4)
- added C84: 22uF, Capacitor_SMD:C_0805_2012Metric_Pad1.18x1.45mm_HandSolder, F.Cu at (114.8, 70.1)
- added C85: 10uF, Capacitor_SMD:C_1206_3216Metric_Pad1.33x1.80mm_HandSolder, F.Cu at (129.2, 119.5)
- added C86: 10uF, Capacitor_SMD:C_1206_3216Metric_Pad1.33x1.80mm_HandSolder, F.Cu at (129.2, 117.1)
- added G***: LOGO, Custom:CoolCube, F.Cu at (153.4, 125.2)
- added J12: SYSTEM CONNECTOR 2, Connector_JST:JST_XH_B8B-XH-A_1x08_P2.50mm_Vertical, F.Cu at (155.9, 115.4)
- added K3: MUTE RELAY, G6K:RELAY_G6K-2P-Y_DC3, F.Cu at (138.4, 118.1)
- added R62: 1K, Resistor_SMD:R_0805_2012Metric_Pad1.20x1.40mm_HandSolder, F.Cu at (143.2, 110.7)
- added R63: 1K, Resistor_SMD:R_0805_2012Metric_Pad1.20x1.40mm_HandSolder, F.Cu at (143.3, 125.2)
- added REF**: KiCad-Logo2_5mm_SilkScreen, Symbol:KiCad-Logo2_5mm_SilkScreen, F.Cu at (156.5, 38.5)
- added TP1: AUDIO IN, TestPoint:TestPoint_Pad_D2.0mm, F.Cu at (143.5, 104.8)
- added U11: OPA134, Package_DIP:DIP-8_W7.62mm_Socket, F.Cu at (114.8, 106.4)
- C27: value 470uF -> 22uF; footprint Capacitor_THT:CP_Radial_D6.3mm_P2.50mm -> Capacitor_THT:CP_Radial_D5.0mm_P2.50mm
- C45: value 10uF -> 22uF
- C58: value 47uF -> 47uF NP
- C64: footprint Capacitor_THT:CP_Radial_D8.0mm_P3.50mm -> Capacitor_THT:CP_Radial_D6.3mm_P2.50mm
- HI-GAIN1: value 10K -> HI-GAIN 10K
- J4: value SYSTEM CONNECTOR -> SYSTEM CONNECTOR 1; footprint Connector_JST:JST_XH_B14B-XH-A_1x14_P2.50mm_Vertical -> Connector_JST:JST_XH_B8B-XH-A_1x08_P2.50mm_Vertical
- K1: value Relay_DPST-NO -> SPK PROTECT
- LO-GAIN1: value 10K -> LOW-GAIN 10K
- U10: value OPA171 -> ULN2003A; footprint Package_SO:SOIC-8_3.9x4.9mm_P1.27mm -> Package_SO:SOIC-16_3.9x9.9mm_P1.27mm
- moved C56 215.1 mm to (191.9, 160.3)
- moved D18 211.5 mm to (182.0, 145.2)
- moved C55 209.2 mm to (185.6, 164.1)
- moved C57 209.0 mm to (185.8, 156.7)
- moved D17 205.2 mm to (176.3, 148.5)
- moved D16 205.2 mm to (176.3, 145.2)
- moved Q5 194.3 mm to (173.7, 130.6)
- moved R42 186.8 mm to (154.3, 169.2), turned to 90 degrees
- moved K1 185.9 mm to (142.4, 155.3)
- moved D2 180.8 mm to (137.2, 154.2), turned to 180 degrees
- moved R49 180.5 mm to (151.6, 137.2)
- moved R53 175.7 mm to (151.6, 134.1)
- moved C54 174.2 mm to (157.0, 176.8), turned to 90 degrees
- moved J10 171.8 mm to (157.5, 162.6), turned to 90 degrees
- moved R46 171.6 mm to (142.7, 137.2)
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Connections:
- net /POWER/PWR-SW renamed /RELAY-SW
- C15 pad 1: Net-(D1-+) -> /RELAY-PWR
- C17 pad 1: Net-(D1-+) -> /RELAY-PWR
- C25 pad 1: /ESPDAC/ESP3V3 -> /ESP3V3
- C45 pad 1: /ESPDAC/ESP3V3 -> /ESP3V3
- C56 pad 2: Net-(D12-A) -> Net-(D14-K)
- C71 pad 1: /ESPDAC/ESP3V3 -> /ESP3V3
- C72 pad 1: /ESPDAC/ESP3V3 -> /ESP3V3
- C77 pad 1: Net-(U10--) -> Net-(U11--)
- D1 pad 4: Net-(D1-+) -> /RELAY-PWR
- D14 pad 1: Net-(D12-A) -> Net-(D14-K)
- D15 pad 1: Net-(D12-A) -> Net-(D14-K)
- D16 pad 1: Net-(D12-A) -> Net-(D14-K)
- IC4 pad 2: /ESPDAC/ESP3V3 -> /ESP3V3
- IC4 pad 6: /ESPDAC/BTN -> /BTN
- J4 pad 1: unconnected-(J4-Pin_1-Pad1) -> /RELAY-PWR
- J4 pad 2: unconnected-(J4-Pin_2-Pad2) -> /ESP3V3
- J4 pad 3: unconnected-(J4-Pin_3-Pad3) -> /BT-LED
- J4 pad 4: unconnected-(J4-Pin_4-Pad4) -> /WIFI-LED
- J4 pad 5: unconnected-(J4-Pin_5-Pad5) -> GND
- J4 pad 6: unconnected-(J4-Pin_6-Pad6) -> /BTN
- J4 pad 7: unconnected-(J4-Pin_7-Pad7) -> /ESP-RX
- J4 pad 8: unconnected-(J4-Pin_8-Pad8) -> /ESP-TX
- J8 pad 3: /ESPDAC/ESP3V3 -> /ESP3V3
- K2 pad 13: Net-(D1-+) -> /RELAY-PWR
- Q3 pad 2: Net-(D12-A) -> Net-(D14-K)
- R1 pad 1: Net-(C1-Pad1) -> /LM1875/HI-IN
- R18 pad 1: /ESPDAC/WIFI-LED -> /WIFI-LED
- R19 pad 1: /ESPDAC/BT-LED -> /BT-LED
- R29 pad 1: /ESPDAC/3V3 -> /ESP3V3
- R30 pad 1: /ESPDAC/3V3 -> /ESP3V3
- R33 pad 2: /LM1875/HI-IN -> Net-(R33-Pad2)
- R34 pad 2: /LM1875/LOW-IN -> Net-(R34-Pad2)
- R49 pad 2: Net-(D12-A) -> Net-(D14-K)
- R7 pad 1: Net-(C7-Pad1) -> /LM1875/LOW-IN
- U10 pad 1: unconnected-(U10-NULL-Pad1) -> Net-(U10-I1)
- U10 pad 2: Net-(U10--) -> unconnected-(U10-I2-Pad2)
- U10 pad 3: Net-(IC6-OUT) -> unconnected-(U10-I3-Pad3)
- U10 pad 4: GND -> unconnected-(U10-I4-Pad4)
- U10 pad 6: Net-(U10--) -> unconnected-(U10-I6-Pad6)
- U10 pad 7: /POWER/12VLIN -> unconnected-(U10-I7-Pad7)
- U10 pad 8: unconnected-(U10-NC-Pad8) -> GND
- U6 pad 2: /ESPDAC/ESP3V3 -> /ESP3V3
- U8 pad 1: /ESPDAC/ESP3V3 -> /ESP3V3
- U8 pad 11: /VOLXOVER/WIPER -> /WIPER
- U8 pad 2: unconnected-(U8-PA4-Pad2) -> Net-(U10-I1)
Routing:
- net /RELAY-SW: track 6.90 -> 303.8 mm, vias 0 -> 1
- net /ESP3V3: track 0.00 -> 138.1 mm, vias 0 -> 6
- net /RELAY-PWR: track 0.00 -> 134.4 mm, vias 0 -> 24
- net /LM1875/LOW-IN: track 0.00 -> 106.6 mm, vias 0 -> 1
- net /LM1875/LOW-OUT: track 17.0 -> 123.1 mm
- net /POWER/-15V: track 14.8 -> 104.4 mm, vias 0 -> 1
- net /LM1875/VCC: track 206.5 -> 295.0 mm, vias 1 -> 4
- net /POWER/12VLIN: track 0.00 -> 76.6 mm, vias 0 -> 3
- net /POWER/+15V: track 10.6 -> 83.1 mm, vias 0 -> 1
- net /BTN: track 0.00 -> 67.9 mm, vias 0 -> 1
- net /BT-LED: track 0.00 -> 66.4 mm, vias 0 -> 1
- net /WIFI-LED: track 0.00 -> 63.6 mm, vias 0 -> 1
- net /LM1875/HI-OUT: track 17.2 -> 77.9 mm
- net /VOLXOVER/LOAD: track 0.00 -> 58.9 mm, vias 0 -> 2
- net /VOLXOVER/CLOCK: track 0.00 -> 56.9 mm, vias 0 -> 2
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- added copper zone on F.Cu, net /POWER/AC
- added copper zone on B.Cu, net /RELAY-PWR
- added copper zone on F.Cu, net /RELAY-PWR
- added copper zone on F.Cu, net Net-(C52-Pad1)
- added copper zone on F.Cu, net Net-(C52-Pad2)
- added copper zone on F.Cu, net Net-(F1-Pad1)
- added copper zone on F.Cu, net Net-(F2-Pad1)
- removed copper zone on F.Cu, net /ESPDAC/ESP3V3
- removed copper zone on B.Cu, net /POWER/AC
- removed copper zone on B.Cu, net Net-(C52-Pad1)
- removed copper zone on B.Cu, net Net-(C52-Pad2)
- removed copper zone on B.Cu, net Net-(D1-+)
- removed copper zone on B.Cu, net Net-(D1--)
- removed copper zone on B.Cu, net Net-(F1-Pad1)
- removed copper zone on B.Cu, net Net-(F2-Pad1)
Other:
- board text added: "ESP-3V3"
- board text added: "ESP-GND"
- board text added: "ESP-RX"
- board text added: "ESP-TX"
- board text added: "LED-3V3"
- board text added: "LED-BT"
- board text added: "LED-WIFI"
- board text added: "LM1875"
- board text added: "MODE-BTN"
- board text added: "MODE-BTN GND"
- board text added: "NC"
- board text added: "P G 3V3"
- board text added: "POWER-SW 1"
- board text added: "POWER-SW 2"
- board text added: "POWER-SW GND"
- board text added: "VCC"
- board text added: "VEE"
- board text added: "VOL-3V3"
- board text added: "VOL-GND"
- board text added: "VOL-WIPER"

Commit message: final design
Parts:
- removed C61, C63: 10uF, Capacitor_SMD:C_1206_3216Metric_Pad1.33x1.80mm_HandSolder
- removed C62: 10nF, Capacitor_SMD:C_0805_2012Metric_Pad1.18x1.45mm_HandSolder
- removed C64: 100uF, Capacitor_THT:CP_Radial_D6.3mm_P2.50mm
- removed C72, C74, C76, C81, C83: 100nF, Capacitor_SMD:C_1206_3216Metric_Pad1.33x1.80mm_HandSolder
- removed C75: 1uF, Capacitor_THT:C_Rect_L7.2mm_W5.5mm_P5.00mm_FKS2_FKP2_MKS2_MKP2
- removed C82: 47uF, Capacitor_THT:CP_Radial_D5.0mm_P2.50mm
- removed IC6: LM1971, Package_SO:SOIC-8_3.9x4.9mm_P1.27mm
- removed IC7: TPS7A4901, Custom:TPS7A4901DRBR
- removed J8: PROG, Connector_JST:JST_XH_B3B-XH-A_1x03_P2.50mm_Vertical
- removed K3: MUTE RELAY, G6K:RELAY_G6K-2P-Y_DC3
- removed R44, R45: 2R2, Resistor_SMD:R_0805_2012Metric_Pad1.20x1.40mm_HandSolder
- removed R48: 432K, Resistor_SMD:R_0805_2012Metric_Pad1.20x1.40mm_HandSolder
- removed R62, R63: 1K, Resistor_SMD:R_0805_2012Metric_Pad1.20x1.40mm_HandSolder
- removed TP1: AUDIO IN, TestPoint:TestPoint_Pad_D2.0mm
- removed U10: ULN2003A, Package_SO:SOIC-16_3.9x9.9mm_P1.27mm
- removed U11: OPA134, Package_DIP:DIP-8_W7.62mm_Socket
- removed U4: PCM5102A, Package_SO:TSSOP-20_4.4x6.5mm_P0.65mm
- removed U8: ATtiny1614, Package_SO:SOIC-14_3.9x8.7mm_P1.27mm
- removed U9: MCP6H01, Package_TO_SOT_SMD:SOT-23-5
- added R64: 1K, Resistor_SMD:R_0805_2012Metric_Pad1.20x1.40mm_HandSolder, F.Cu at (59.4, 105.2)
- added U12: PCM5122PW, Package_SO:TSSOP-28_4.4x9.7mm_P0.65mm, F.Cu at (98.9, 114.0)
- C33: value 1uF -> 10uF
- C60: value 10nF -> 100nF; footprint Capacitor_SMD:C_0805_2012Metric_Pad1.18x1.45mm_HandSolder -> Capacitor_SMD:C_1206_3216Metric_Pad1.33x1.80mm_HandSolder
- J10: value LOW OUT -> HI OUT
- J7: value HI OUT -> LOW OUT
- R47: value 49K9 -> 10K; footprint Resistor_SMD:R_0805_2012Metric_Pad1.20x1.40mm_HandSolder -> Resistor_SMD:R_0603_1608Metric_Pad0.98x0.95mm_HandSolder
- R59, R60: value 10K -> 4K7
- moved C57 141.3 mm to (47.7, 127.3)
- moved D18 137.9 mm to (44.7, 132.9), turned to 90 degrees
- moved C56 130.6 mm to (64.7, 130.7)
- moved C55 124.0 mm to (64.7, 136.5)
- moved Q5 117.8 mm to (56.0, 132.8)
- moved D3 116.4 mm to (147.3, 27.3), turned to 180 degrees
- moved J12 108.5 mm to (48.8, 98.7), turned to -90 degrees
- moved D17 106.6 mm to (70.3, 136.9), turned to -90 degrees
- moved C41 104.8 mm to (151.6, 80.3)
- moved C42 104.8 mm to (134.1, 80.3)
- moved C59 104.8 mm to (147.1, 80.1)
- moved C65 104.8 mm to (140.1, 79.1)
- moved C70 104.8 mm to (144.5, 68.9)
- moved C78 104.8 mm to (138.5, 75.8)
- moved C80 104.8 mm to (140.6, 69.7)
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Connections:
- C27 pad 1: Net-(IC3-OUT) -> /ESPDAC/AVDD
- C28 pad 1: Net-(IC3-OUT) -> /ESPDAC/AVDD
- C31 pad 1: Net-(IC3-OUT) -> /ESPDAC/AVDD
- C35 pad 1: Net-(IC3-OUT) -> /ESPDAC/AVDD
- C60 pad 1: Net-(IC7-NR/SS) -> Net-(IC4-IO35)
- C68 pad 1: /ESPDAC/CPVDD -> /ESPDAC/AVDD
- C69 pad 1: /ESPDAC/CPVDD -> /ESPDAC/AVDD
- C77 pad 1: Net-(U11--) -> /ESPDAC/MONO-OUT
- IC3 pad 5: Net-(IC3-OUT) -> /ESPDAC/AVDD
- IC4 pad 33: unconnected-(IC4-IO21-Pad33) -> /ESPDAC/SDA
- IC4 pad 36: unconnected-(IC4-IO22-Pad36) -> /ESPDAC/SCL
- IC4 pad 7: unconnected-(IC4-IO35-Pad7) -> Net-(IC4-IO35)
- J10 pad 1: Net-(J10-P1-Pad1) -> Net-(C58-Pad1)
- J10 pad 2: Net-(J10-P1-Pad1) -> Net-(C58-Pad1)
- J7 pad 1: Net-(C58-Pad1) -> Net-(J7-P1-Pad1)
- J7 pad 2: Net-(C58-Pad1) -> Net-(J7-P1-Pad1)
- K1 pad 24: Net-(J10-P1-Pad1) -> Net-(J7-P1-Pad1)
- R33 pad 2: Net-(R33-Pad2) -> /LM1875/HI-IN
- R34 pad 2: Net-(R34-Pad2) -> /LM1875/LOW-IN
- R47 pad 1: Net-(IC7-FB) -> /ESP3V3
- R47 pad 2: GND -> /BTN
- R59 pad 1: Net-(U9-+) -> /ESP3V3
- R59 pad 2: GND -> /ESPDAC/SDA
- R60 pad 1: /POWER/12VLIN -> /ESP3V3
- R60 pad 2: Net-(U9-+) -> /ESPDAC/SCL
Routing:
- net /LM1875/VCC: track 295.0 -> 412.2 mm, vias 4 -> 2
- net /RELAY-SW: track 303.8 -> 199.4 mm, vias 1 -> 0
- net /POWER/12VLIN: track 76.6 -> 0.00 mm, vias 3 -> 0
- net /LM1875/LOW-OUT: track 123.1 -> 57.4 mm
- net /VOLXOVER/LOAD: track 58.9 -> 0.00 mm, vias 2 -> 0
- net /BT-LED: track 66.4 -> 9.01 mm, vias 1 -> 0
- net /VOLXOVER/CLOCK: track 56.9 -> 0.00 mm, vias 2 -> 0
- net /VOLXOVER/DATA: track 56.6 -> 0.00 mm, vias 2 -> 0
- net /RELAY-PWR: track 134.4 -> 190.3 mm, vias 24 -> 1
- net /WIFI-LED: track 63.6 -> 8.92 mm, vias 1 -> 0
- net Net-(IC4-IO35): track 0.00 -> 52.2 mm
- net /POWER/AC: track 0.00 -> 51.8 mm
- net /ESPDAC/AVDD: track 0.00 -> 50.4 mm, vias 0 -> 5
- net Net-(IC4-IO33): track 4.68 -> 54.2 mm, vias 0 -> 2
- net Net-(IC4-IO32): track 6.46 -> 50.2 mm, vias 0 -> 2
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- added copper zone on B.Cu, net /POWER/AC
- added copper zone on B.Cu, net GND
- added copper zone on B.Cu, net Net-(C52-Pad1)
- added copper zone on B.Cu, net Net-(C52-Pad2)
- added copper zone on B.Cu, net Net-(D1--)
- added copper zone on B.Cu, net Net-(F1-Pad1)
- added copper zone on B.Cu, net Net-(F2-Pad1)
- removed copper zone on F.Cu, net /RELAY-PWR
- removed copper zone on F.Cu, net Net-(C52-Pad1)
- removed copper zone on F.Cu, net Net-(C52-Pad2)
- removed copper zone on F.Cu, net Net-(D1--)
- removed copper zone on F.Cu, net Net-(F1-Pad1)
- removed copper zone on F.Cu, net Net-(F2-Pad1)
Other:
- board size 120 x 168.9 mm -> 120 x 142 mm
- board text added: "Bi-Amped LM1875 System SnapCast/Bluetooth PCM5122 ±25V Tom Watson Audio 2026"
- board text removed: "Bi-Amped LM1875 System SnapCast/Bluetooth PCM5102 ±25V Tom Watson Audio 2026"
- board text removed: "P G 3V3"

Commit message: more
Parts:
- moved G*** 121.4 mm to (127.8, 113.9)
Changed lines of the file:
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@@
 			(drillshape 0)
 			(scaleselection 1)
-			(outputdirectory "/Users/tomwatson/Documents/")
+			(outputdirectory "/Users/tomwatson/Desktop/Gerber files/LM1875Cube/")
 		)
 	)
@@
 	(footprint "Custom:LOGONEW"
 		(layer "F.Cu")
-		(at 155.448 -4.318)
+		(at 127.762 113.919)
 		(property "Reference" "G***"
 			(at 0 0 0)
