File: CoolCubeLM1875kicad_pro/CoolCubeLM1875kicad_pro.kicad_sch (KiCad schematic)
At the start: 7 parts, among them J4 SYSTEM CONNECTOR

Commit message: more work
Parts:
- removed J4: SYSTEM CONNECTOR, Connector_JST:JST_XH_B14B-XH-A_1x14_P2.50mm_Vertical, symbol Connector:Conn_01x14_Socket
- added J12: SYSTEM CONNECTOR 2, Connector_JST:JST_XH_B8B-XH-A_1x08_P2.50mm_Vertical, symbol Connector:Conn_01x08_Socket
- added J4: SYSTEM CONNECTOR 1, Connector_JST:JST_XH_B8B-XH-A_1x08_P2.50mm_Vertical, symbol Connector:Conn_01x08_Socket
Connections:
- net ESP-RX: now also J4.7 (Pin_7)
- net ESP-TX: now also J4.8 (Pin_8)
- new net BT-LED: J4.3 (Pin_3)
- new net BTN: J4.6 (Pin_6)
- new net ESP3V3: J12.5 (Pin_5), J12.7 (Pin_7), J4.2 (Pin_2)
- new net GND: J12.2 (Pin_2), J12.3 (Pin_3), J12.8 (Pin_8), J4.5 (Pin_5)
- new net RELAY-PWR: J4.1 (Pin_1)
- new net RELAY-SW: J12.6 (Pin_6)
- new net WIFI-LED: J4.4 (Pin_4)
- new net WIPER: J12.4 (Pin_4)
Other:
- sheet POWER ports: added RELAT-SW, RELAY-PWR; removed PWR-SW
- sheet VOLXOVER ports: added 5VBUCK; removed none

Commit message: final design
Other:
- sheet ESPDAC ports: added WIPER; removed none
- sheet POWER ports: added none; removed 12VLIN
- sheet VOLXOVER ports: added none; removed 12VLDO, 5VBUCK, PROG, WIPER
Changed lines of the file:
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@@
-	)
-	(junction
-		(at 156.21 115.57)
-		(diameter 0)
-		(color 0 0 0 0)
 	)
 	(junction
@@
 	(wire
 		(pts
+			(xy 102.87 128.27) (xy 111.76 128.27)
+		)
+		(stroke
+			(width 0)
+			(type default)
+		)
+	)
+	(wire
+		(pts
 			(xy 199.39 39.37) (xy 199.39 48.26)
 		)
@@
 	(wire
 		(pts
-			(xy 199.39 66.04) (xy 208.28 66.04)
-		)
-		(stroke
-			(width 0)
-			(type default)
-		)
-	)
-	(wire
-		(pts
 			(xy 241.3 39.37) (xy 199.39 39.37)
 		)
@@
 	(wire
 		(pts
-			(xy 209.55 111.76) (xy 209.55 82.55)
-		)
-		(stroke
-			(width 0)
-			(type default)
-		)
-	)
-	(wire
-		(pts
 			(xy 226.06 116.84) (xy 251.46 116.84)
 		)
@@
 	(wire
 		(pts
-			(xy 199.39 82.55) (xy 199.39 66.04)
-		)
-		(stroke
-			(width 0)
-			(type default)
-		)
-	)
-	(wire
-		(pts
 			(xy 214.63 85.09) (xy 214.63 109.22)
 		)
@@
 	(wire
 		(pts
-			(xy 209.55 82.55) (xy 199.39 82.55)
-		)
-		(stroke
-			(width 0)
-			(type default)
-		)
-	)
-	(wire
-		(pts
 			(xy 153.67 99.06) (xy 153.67 109.22)
 		)
@@
 	(wire
 		(pts
-			(xy 199.39 129.54) (xy 205.74 129.54)
-		)
-		(stroke
-			(width 0)
-			(type default)
-		)
-	)
-	(wire
-		(pts
 			(xy 111.76 66.04) (xy 101.6 66.04)
 		)
@@
 	(wire
 		(pts
-			(xy 199.39 111.76) (xy 209.55 111.76)
-		)
-		(stroke
-			(width 0)
-			(type default)
-		)
-	)
-	(wire
-		(pts
 			(xy 176.53 48.26) (xy 176.53 20.32)
 		)
@@
 		(pts
 			(xy 204.47 146.05) (xy 204.47 158.75)
-		)
-		(stroke
-			(width 0)
-			(type default)
-		)
-	)
-	(wire
-		(pts
-			(xy 156.21 115.57) (xy 163.83 115.57)
 		)
 		(stroke
@@
 	)
 	(label "WIPER"
-		(at 205.74 129.54 0)
-		(effects
-			(font
-				(size 1.27 1.27)
-			)
-			(justify left bottom)
+		(at 102.87 128.27 180)
+		(effects
+			(font
+				(size 1.27 1.27)
+			)
+			(justify right bottom)
 		)
 	)
@@
 			)
 		)
+		(pin "WIPER" input
+			(at 111.76 128.27 180)
+			(effects
+				(font
+					(size 1.27 1.27)
+				)
+				(justify left)
+			)
+		)
 		(instances
 			(project "CoolCubeLM1875kicad_pro"
@@
 			)
 		)
-		(pin "12VLIN" input
-			(at 208.28 66.04 180)
-			(effects
-				(font
-					(size 1.27 1.27)
-				)
-				(justify left)
-			)
-		)
 		(pin "AC" input
 			(at 240.03 55.88 0)
@@
 			)
 		)
-		(pin "12VLDO" input
-			(at 199.39 111.76 0)
-			(effects
-				(font
-					(size 1.27 1.27)
-				)
-				(justify right)
-			)
-		)
-		(pin "PROG" input
-			(at 199.39 127 0)
-			(effects
-				(font
-					(size 1.27 1.27)
-				)
-				(justify right)
-			)
-		)
-		(pin "WIPER" input
-			(at 199.39 129.54 0)
-			(effects
-				(font
-					(size 1.27 1.27)
-				)
-				(justify right)
-			)
-		)
 		(pin "ESP3V3" input
 			(at 163.83 109.22 180)
 			(effects
 				(font
-					(size 1.27 1.27)
-				)
-				(justify left)
-			)
-		)
-		(pin "5VBUCK" input
-			(at 163.83 115.57 180)
-			(effects
-				(font
