File: CoolCubeLM1875kicad_pro/ESPDAC.kicad_sch (KiCad schematic)
At the start: 41 parts, among them IC2 RESET, IC3 TPS7A2033, IC4 ESP32-Wrover-IE-N16R8, IC5 BOOT, U4 PCM5102A, U6 AMS1117-3.3

Commit message: more work
Parts:
- added C84: 22uF, Capacitor_SMD:C_0805_2012Metric_Pad1.18x1.45mm_HandSolder, symbol Device:C
- added TP1: AUDIO IN, TestPoint:TestPoint_Pad_D2.0mm, symbol Connector:TestPoint
- C27: value 470uF -> 22uF; footprint Capacitor_THT:CP_Radial_D6.3mm_P2.50mm -> Capacitor_THT:CP_Radial_D5.0mm_P2.50mm
- C45: value 10uF -> 22uF
Connections:
- net 3V3 is gone; now on net ESP3V3: R29.1, R30.1
- net ESP5V: now also C84.1
- net GND: now also C84.2
- net MONO-OUT: now also TP1.1

Commit message: final design
Parts:
- removed R44, R45: 2R2, Resistor_SMD:R_0805_2012Metric_Pad1.20x1.40mm_HandSolder, symbol Device:R
- removed TP1: AUDIO IN, TestPoint:TestPoint_Pad_D2.0mm, symbol Connector:TestPoint
- removed U4: PCM5102A, Package_SO:TSSOP-20_4.4x6.5mm_P0.65mm, symbol Audio:PCM5102A
- added C60: 100nF, Capacitor_SMD:C_1206_3216Metric_Pad1.33x1.80mm_HandSolder, symbol Device:C
- added R47: 10K, Resistor_SMD:R_0603_1608Metric_Pad0.98x0.95mm_HandSolder, symbol Device:R
- added R59, R60: 4K7, Resistor_SMD:R_0805_2012Metric_Pad1.20x1.40mm_HandSolder, symbol Device:R
- added R64: 1K, Resistor_SMD:R_0805_2012Metric_Pad1.20x1.40mm_HandSolder, symbol Device:R
- added U12: PCM5122PW, Package_SO:TSSOP-28_4.4x9.7mm_P0.65mm, symbol Audio:PCM5122PW
- C33: value 1uF -> 10uF
Connections:
- net CPVDD is gone; now on net AVDD: C68.1, C69.1
- net AVDD: now also C27.1, C28.1, C31.1, C35.1, IC3.5 (OUT), U12.1 (CPVDD), U12.28 (DVDD), U12.8 (AVDD)
- net BCK: now also U12.21 (BCK)
- net BTN: now also R47.2
- net DOUT: now also U12.22 (DIN)
- net ESP3V3: now also R47.1, R59.1, R60.1
- net GND: now also C60.2, U12.27 (DGND), U12.3 (CPGND), U12.9 (AGND)
- net LRCK: now also U12.23 (LRCK)
- net at C32.1, C33.1: now also U12.26 (LDOO)
- net at C30.1: now also U12.2 (CAPP)
- net at C30.2: now also U12.4 (CAPM)
- net at C29.1: now also U12.5 (VNEG)
- net at R31.1: now also U12.6 (OUTL)
- net at R32.2: now also U12.7 (OUTR)
- net SDA: now reaches IC4.33 (IO21)
- net SDA: now also R59.2, U12.11 (SDA/MOSI/ATT2)
- net SCL: now reaches IC4.36 (IO22)
- net SCL: now also R60.2, U12.12 (SCL/MC/ATT1)
- net at IC4.7 (IO35): now also C60.1, R64.2
- new net WIPER: R64.1
Other:
- moved on the sheet: C29, C30, C32, C33
