File: CoolCubeLM1875kicad_pro/LM1875.kicad_sch (KiCad schematic)
At the start: 28 parts, among them U1 LM1875, U2 LM1875

Commit message: more work
Parts:
- removed C1, C7: 1uF, Capacitor_THT:C_Rect_L7.5mm_W6.5mm_P5.00mm, symbol Device:C
Connections:
- net HI-IN: now also R1.1
- net LOW-IN: now also R7.1
Changed lines of the file:
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@@
-	(wire
-		(pts
-			(xy 43.18 99.06) (xy 46.99 99.06)
-		)
-		(stroke
-			(width 0)
-			(type default)
-		)
-	)
 	(wire
 		(pts
@@
 	(wire
 		(pts
-			(xy 43.18 33.02) (xy 46.99 33.02)
-		)
-		(stroke
-			(width 0)
-			(type default)
-		)
-	)
-	(wire
-		(pts
 			(xy 139.7 101.6) (xy 118.11 101.6)
 		)
@@
 	(wire
 		(pts
-			(xy 27.94 33.02) (xy 35.56 33.02)
+			(xy 35.56 33.02) (xy 46.99 33.02)
 		)
 		(stroke
@@
 	(wire
 		(pts
-			(xy 27.94 99.06) (xy 35.56 99.06)
+			(xy 35.56 99.06) (xy 46.99 99.06)
 		)
 		(stroke
@@
 	(hierarchical_label "LOW-IN"
 		(shape input)
-		(at 27.94 99.06 180)
+		(at 35.56 99.06 180)
 		(effects
 			(font
@@
 	(hierarchical_label "HI-IN"
 		(shape input)
-		(at 27.94 33.02 180)
+		(at 35.56 33.02 180)
 		(effects
 			(font
@@
 				(path "/d273928c-b496-49db-97f0-9ad0f6f64c23/af254f73-3587-4e22-8e81-792d39ee5b44"
 					(reference "R1")
-					(unit 1)
-				)
-			)
-		)
-	)
-	(symbol
-		(lib_id "Device:C")
-		(at 39.37 33.02 270)
-		(unit 1)
-		(exclude_from_sim no)
-		(in_bom yes)
-		(on_board yes)
-		(dnp no)
-		(fields_autoplaced yes)
-		(property "Reference" "C1"
-			(at 39.37 25.4 90)
-			(effects
-				(font
-					(size 1.27 1.27)
-				)
-			)
-		)
-		(property "Value" "1uF"
-			(at 39.37 27.94 90)
-			(effects
-				(font
-					(size 1.27 1.27)
-				)
-			)
-		)
-		(property "Footprint" "Capacitor_THT:C_Rect_L7.5mm_W6.5mm_P5.00mm"
-			(at 35.56 33.9852 0)
-			(effects
-				(font
-					(size 1.27 1.27)
-				)
-				(hide yes)
-			)
-		)
-		(property "Datasheet" "~"
-			(at 39.37 33.02 0)
-			(effects
-				(font
-					(size 1.27 1.27)
-				)
-				(hide yes)
-			)
-		)
-		(property "Description" "Unpolarized capacitor"
-			(at 39.37 33.02 0)
-			(effects
-				(font
-					(size 1.27 1.27)
-				)
-				(hide yes)
-			)
-		)
-		(pin "2"
-		)
-		(pin "1"
-		)
-		(instances
-			(project "CoolCubeLM1875kicad_pro"
-				(path "/d273928c-b496-49db-97f0-9ad0f6f64c23/af254f73-3587-4e22-8e81-792d39ee5b44"
-					(reference "C1")
 					(unit 1)
 				)
@@
 					(unit 1)
 				)
-			)
-		)
-	)
-	(symbol
-		(lib_id "Device:C")
-		(at 39.37 99.06 270)
-		(unit 1)
-		(exclude_from_sim no)
-		(in_bom yes)
-		(on_board yes)
-		(dnp no)
-		(fields_autoplaced yes)
-		(property "Reference" "C7"
-			(at 39.37 91.44 90)
-			(effects
-				(font
-					(size 1.27 1.27)
-				)
-			)
-		)
-		(property "Value" "1uF"
-			(at 39.37 93.98 90)
-			(effects
-				(font
-					(size 1.27 1.27)
-				)
-			)
-		)
-		(property "Footprint" "Capacitor_THT:C_Rect_L7.5mm_W6.5mm_P5.00mm"
-			(at 35.56 100.0252 0)
-			(effects
-				(font
-					(size 1.27 1.27)
-				)
-				(hide yes)
-			)
-		)
-		(property "Datasheet" "~"
-			(at 39.37 99.06 0)
-			(effects
-				(font
-					(size 1.27 1.27)
-				)
-				(hide yes)
-			)
-		)
-		(property "Description" "Unpolarized capacitor"
-			(at 39.37 99.06 0)
-			(effects
-				(font
-					(size 1.27 1.27)
-				)
-				(hide yes)
-			)
-		)
-		(pin "2"
-		)
-		(pin "1"
-		)
-		(instances
-			(project "CoolCubeLM1875kicad_pro"
-				(path "/d273928c-b496-49db-97f0-9ad0f6f64c23/af254f73-3587-4e22-8e81-792d39ee5b44"
-					(reference "C7")
-					(unit 1)
-				)
