File: CoolCubeLM1875kicad_pro/POWER.kicad_sch (KiCad schematic)
At the start: 46 parts, among them IC7 TPS7A4901, J1 AC, J2 AC, J3 GND, J5 GND, J6 GND, K2 STBY RELAY, U3 LMR51430, U7 TPS7A39

Commit message: more work
Parts:
- added J9: GND, Spade connector:TE_62409-1, symbol Spade connector:62409-1
- C64: footprint Capacitor_THT:CP_Radial_D8.0mm_P3.50mm -> Capacitor_THT:CP_Radial_D6.3mm_P2.50mm
Connections:
- net GND: now also J9.1 (P1), J9.2 (P1)
- net RELAY-PWR: now reaches C15.1, C17.1, D1.4 (+), K2.13
- net PWR-SW renamed RELAT-SW

Commit message: final design
Parts:
- removed C60, C62: 10nF, Capacitor_SMD:C_0805_2012Metric_Pad1.18x1.45mm_HandSolder, symbol Device:C
- removed C61, C63: 10uF, Capacitor_SMD:C_1206_3216Metric_Pad1.33x1.80mm_HandSolder, symbol Device:C
- removed C64: 100uF, Capacitor_THT:CP_Radial_D6.3mm_P2.50mm, symbol Device:C_Polarized
- removed IC7: TPS7A4901, Custom:TPS7A4901DRBR, symbol Custom:TPS7A4901DRBR
- removed R47: 49K9, Resistor_SMD:R_0805_2012Metric_Pad1.20x1.40mm_HandSolder, symbol Device:R
- removed R48: 432K, Resistor_SMD:R_0805_2012Metric_Pad1.20x1.40mm_HandSolder, symbol Device:R

Commit message: more
Parts:
- J1, J2, J3, J5, J6, J9: footprint Spade connector:TE_62409-1 -> (none)
