File: CoolCubeLM1875kicad_pro/RELAY.kicad_sch (KiCad schematic)
At the start: 31 parts, among them J10 LOW OUT, J7 HI OUT, K1 Relay_DPST-NO, Q2 BD140, Q3 BC549, Q4 BC559, Q5 BC549

Commit message: more work
Parts:
- C58: value 47uF -> 47uF NP
- K1: value Relay_DPST-NO -> SPK PROTECT
Connections:
- net at C56.2, D14.1 (K), D15.1 (K)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: no longer D12.2 (A), D13.2 (A), D17.2 (A), Q3.3 (E)
- new net: D12.2 (A), D13.2 (A), D17.2 (A), Q3.3 (E)
Changed lines of the file:
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@@
-	)
-	(junction
-		(at 80.01 114.3)
-		(diameter 0)
-		(color 0 0 0 0)
 	)
 	(junction
@@
 	(wire
 		(pts
-			(xy 80.01 114.3) (xy 72.39 114.3)
+			(xy 72.39 114.3) (xy 118.11 114.3)
 		)
 		(stroke
@@
 	(wire
 		(pts
-			(xy 80.01 114.3) (xy 118.11 114.3)
-		)
-		(stroke
-			(width 0)
-			(type default)
-		)
-	)
-	(wire
-		(pts
 			(xy 142.24 62.23) (xy 142.24 67.31)
 		)
@@
 	(wire
 		(pts
-			(xy 80.01 88.9) (xy 80.01 114.3)
-		)
-		(stroke
-			(width 0)
-			(type default)
-		)
-	)
-	(wire
-		(pts
 			(xy 118.11 52.07) (xy 134.62 52.07)
 		)
@@
 	(wire
 		(pts
-			(xy 80.01 124.46) (xy 80.01 114.3)
-		)
-		(stroke
-			(width 0)
-			(type default)
-		)
-	)
-	(wire
-		(pts
 			(xy 63.5 27.94) (xy 80.01 27.94)
 		)
@@
 		(pts
 			(xy 231.14 83.82) (xy 231.14 96.52)
+		)
+		(stroke
+			(width 0)
+			(type default)
+		)
+	)
+	(wire
+		(pts
+			(xy 80.01 88.9) (xy 80.01 124.46)
 		)
 		(stroke
@@
 			)
 		)
-		(property "Value" "47uF"
+		(property "Value" "47uF NP"
 			(at 264.16 74.9299 0)
 			(effects
@@
 			)
 		)
-		(property "Value" "Relay_DPST-NO"
+		(property "Value" "SPK PROTECT"
 			(at 240.03 99.06 90)
 			(effects

Commit message: final design
Parts:
- J10: value LOW OUT -> HI OUT
- J7: value HI OUT -> LOW OUT
Connections:
- net at J7.1 (P1), J7.2 (P1): now also K1.24; no longer C58.1
- net at J10.1 (P1), J10.2 (P1): now also C58.1; no longer K1.24
Other:
- moved on the sheet: C58, J10, J7

Commit message: more
Parts:
- J10, J7: footprint Spade connector:TE_62409-1 -> (none)
