File: CoolCubeLM1875kicad_pro/VOLXOVER.kicad_sch (KiCad schematic)
At the start: 43 parts, among them IC6 LM1971, J8 PROG, U10 OPA171, U5 OPA1656ID, U8 ATtiny1614, U9 MCP6H01

Commit message: more work
Parts:
- removed U10: OPA171, Package_SO:SOIC-8_3.9x4.9mm_P1.27mm, symbol Amplifier_Operational:TL081
- added C85, C86: 10uF, Capacitor_SMD:C_1206_3216Metric_Pad1.33x1.80mm_HandSolder, symbol Device:C
- added K3: MUTE RELAY, G6K:RELAY_G6K-2P-Y_DC3, symbol G6K-2P-Y:G6K-2P-Y_DC3
- added R62, R63: 1K, Resistor_SMD:R_0805_2012Metric_Pad1.20x1.40mm_HandSolder, symbol Device:R
- added U10: ULN2003A, Package_SO:SOIC-16_3.9x9.9mm_P1.27mm, symbol Transistor_Array:ULN2003A
- added U11: OPA134, Package_DIP:DIP-8_W7.62mm_Socket, symbol Amplifier_Operational:OPA134
- HI-GAIN1: value 10K -> HI-GAIN 10K
- LO-GAIN1: value 10K -> LOW-GAIN 10K
Connections:
- net +15V: now also C85.1
- net -15V: now also C86.2
- net 12VLDO: now also U11.7 (V+)
- net GND: now also C85.2, C86.1, K3.2, K3.7, U10.8 (GND), U11.4 (V-)
- net OUT-HI: now also K3.3, R62.2; no longer R33.2
- net OUT-LOW: now also K3.6, R63.2; no longer R34.2
- net at C77.1: now also U11.2 (-), U11.6
- net at IC6.2 (OUT): now also U11.3 (+)
- net at U8.2 (PA4): now also U10.1 (I1)
- new net: R34.2, R63.1
- new net: R33.2, R62.1
- new net 5VBUCK: U10.9 (COM)
Other:
- moved on the sheet: C71, C72, J8, R33, R34, U8

Commit message: final design
Parts:
- removed C71: 10uF, Capacitor_THT:CP_Radial_D4.0mm_P1.50mm, symbol Device:C_Polarized
- removed C72, C74, C76, C81, C83: 100nF, Capacitor_SMD:C_1206_3216Metric_Pad1.33x1.80mm_HandSolder, symbol Device:C
- removed C75: 1uF, Capacitor_THT:C_Rect_L7.2mm_W5.5mm_P5.00mm_FKS2_FKP2_MKS2_MKP2, symbol Device:C
- removed C82: 47uF, Capacitor_THT:CP_Radial_D5.0mm_P2.50mm, symbol Device:C_Polarized
- removed IC6: LM1971, Package_SO:SOIC-8_3.9x4.9mm_P1.27mm, symbol Custom:LM1971MX_NOPB
- removed J8: PROG, Connector_JST:JST_XH_B3B-XH-A_1x03_P2.50mm_Vertical, symbol Connector:Conn_01x03_Socket
- removed K3: MUTE RELAY, G6K:RELAY_G6K-2P-Y_DC3, symbol G6K-2P-Y:G6K-2P-Y_DC3
- removed R59, R60: 10K, Resistor_SMD:R_0805_2012Metric_Pad1.20x1.40mm_HandSolder, symbol Device:R
- removed R62, R63: 1K, Resistor_SMD:R_0805_2012Metric_Pad1.20x1.40mm_HandSolder, symbol Device:R
- removed U10: ULN2003A, Package_SO:SOIC-16_3.9x9.9mm_P1.27mm, symbol Transistor_Array:ULN2003A
- removed U11: OPA134, Package_DIP:DIP-8_W7.62mm_Socket, symbol Amplifier_Operational:OPA134
- removed U8: ATtiny1614, Package_SO:SOIC-14_3.9x8.7mm_P1.27mm, symbol MCU_Microchip_ATtiny:ATtiny1614-SS
- removed U9: MCP6H01, Package_TO_SOT_SMD:SOT-23-5, symbol Amplifier_Operational:MCP6001-OT
Connections:
- net MONO-IN: now also C77.1
- net OUT-HI: now also R33.2
- net OUT-LOW: now also R34.2
Other:
- moved on the sheet: C41, C42, C43, C77, C85, C86, U5C
